Commit message: Spinning arms from parallel processes

File: robot/robot.urdf (robot description, URDF)
Before this commit: robot onshape, 8 links, 7 joints
Links:
- added link part_2_1, mass 1e-9
- added link part_2_1_0_part_2, mass 0; collision mesh filename=package://part_2.stl; visual mesh filename=package://part_2.stl
- added link part_3_1, mass 1e-9
- added link part_3_1_0_part_3, mass 0; collision mesh filename=package://part_3.stl; visual mesh filename=package://part_3.stl
- added link part_4_1, mass 1e-9
- added link part_4_1_0_part_4, mass 0; collision mesh filename=package://part_4.stl; visual mesh filename=package://part_4.stl
- link torso_1_0_torso: mass 0 -> 29.6172
Joints:
- removed joint distal
- removed joint proximal
- removed joint shoulder
- added joint distal_left: type revolute, parent part_3_1, child part_4_1, origin xyz=0.193394 -0.0097 0.166524 rpy=1.66533e-16 -7.21645e-16 3.88578e-16, axis 0 -1 0, limit effort=1.5 velocity=22
- added joint distal_right: type revolute, parent part_6_1, child part_7_1, origin xyz=-0.193394 -0.0097 0.166524 rpy=2.01609e-16 0.811584 -3.32655e-15, axis 0 -1 0, limit effort=1.5 velocity=22
- added joint part_2_1_part_2_1_0_part_2_fixing: type fixed, parent part_2_1, child part_2_1_0_part_2, origin xyz=-0.13182 5.55112e-17 -0.303536 rpy=-5.55112e-17 -0 0, axis 0 0 0
- added joint part_3_1_part_3_1_0_part_3_fixing: type fixed, parent part_3_1, child part_3_1_0_part_3, origin xyz=-0.119445 -1.38778e-17 -0.344194 rpy=-5.55112e-17 -0 0, axis 0 0 0
- added joint part_4_1_part_4_1_0_part_4_fixing: type fixed, parent part_4_1, child part_4_1_0_part_4, origin xyz=-0.312839 0.0075 -0.510718 rpy=0 -0 5.55112e-17, axis 0 0 0
- added joint proximal_left: type revolute, parent part_2_1, child part_3_1, origin xyz=-0.0141421 0 0.0424264 rpy=-7.77156e-16 7.77156e-16 5.55112e-17, axis -0.707107 0 0.707107, limit effort=1.5 velocity=22
- added joint proximal_right: type revolute, parent part_5_1, child part_6_1, origin xyz=0.0141421 -4.16334e-17 0.0424264 rpy=-0.705905 -0.269757 -0.705905, axis 0.707107 0 0.707107, limit effort=1.5 velocity=22
- added joint shoulder_left: type revolute, parent torso_1, child part_2_1, origin xyz=0.13182 -2.77556e-17 0.303536 rpy=-0.752186 -0.309384 -0.752186, axis 0.707107 0 0.707107, limit effort=1.5 velocity=22
- added joint shoulder_right: type revolute, parent torso_1, child part_5_1, origin xyz=-0.13182 -2.77556e-17 0.303536 rpy=-0.706606 0.270333 0.706606, axis 0.707107 0 -0.707107, limit effort=1.5 velocity=22

Commit message: Improved pose tracking with proper transforms

File: robot/robot.urdf (robot description, URDF)
Before this commit: robot onshape, 14 links, 13 joints
Links:
- added link part_4_2, mass 1e-9
- added link part_4_2_0_part_4, mass 0; collision mesh filename=package://part_4.stl; visual mesh filename=package://part_4.stl
- added link part_7_2, mass 1e-9
- added link part_7_2_0_part_7, mass 0; collision mesh filename=package://part_7.stl; visual mesh filename=package://part_7.stl
Joints:
- added joint left_tip: type revolute, parent part_4_1, child part_4_2, origin xyz=-0.0431288 0.0075 -0.133191 rpy=0 -3.33067e-16 -1.11022e-16, axis 0 1 0, limit effort=1.5 velocity=22
- added joint part_4_2_part_4_2_0_part_4_fixing: type fixed, parent part_4_2, child part_4_2_0_part_4, origin xyz=-0.235057 -0.0075 -0.432936 rpy=5.55112e-17 -0 5.55112e-17, axis 0 0 0
- added joint part_7_2_part_7_2_0_part_7_fixing: type fixed, parent part_7_2, child part_7_2_0_part_7, origin xyz=0.235057 0.0075 -0.432936 rpy=0 -0 1.38778e-17, axis 0 0 0
- added joint right_tip: type revolute, parent part_7_1, child part_7_2, origin xyz=0.0431288 0.0075 -0.133191 rpy=-2.77556e-17 5.55112e-17 -7.84095e-15, axis 0 -1 0, limit effort=1.5 velocity=22
- joint distal_left: origin xyz=0.193394 -0.0097 0.166524 rpy=1.66533e-16 -7.21645e-16 3.88578e-16 -> xyz=0.115612 -0.0097 0.0887419 rpy=1.66533e-16 -7.21645e-16 3.88578e-16
- joint distal_right: origin xyz=-0.193394 -0.0097 0.166524 rpy=2.01609e-16 0.811584 -3.32655e-15 -> xyz=-0.115612 -0.0097 0.0887419 rpy=4.03219e-17 0.811584 -3.72977e-15
- joint part_4_1_part_4_1_0_part_4_fixing: origin xyz=-0.312839 0.0075 -0.510718 rpy=0 -0 5.55112e-17 -> xyz=-0.235057 0.0075 -0.432936 rpy=0 -0 5.55112e-17
- joint part_7_1_part_7_1_0_part_7_fixing: origin xyz=0.312839 0.0075 -0.510718 rpy=-2.77556e-17 5.55112e-17 1.38778e-17 -> xyz=0.235057 0.0075 -0.432936 rpy=5.55112e-17 -0 4.16334e-17
